Commit message: perf: add black tape on gripper'sfinger

File: urdf/umi_gripper/umi_gripper.urdf (robot description, URDF)
Before this commit: robot umi_gripper, 19 links, 18 joints
Links:
- added link left_tape, mass 0.005; visual box size=0.12 0.0258 0.00002
- added link right_tape, mass 0.005; visual box size=0.12 0.0258 0.00002
Joints:
- added joint fix_left_tape_and_left_finger: type fixed, parent left_finger, child left_tape, origin xyz=0 0 0 rpy=0 0 0
- added joint fix_right_tape_and_right_finger: type fixed, parent right_finger, child right_tape, origin xyz=0 0 0 rpy=0 0 0

Commit message: perf: add empty eef_link (unify name)

File: urdf/umi_gripper/umi_gripper.urdf (robot description, URDF)
Before this commit: robot umi_gripper, 21 links, 20 joints
Links:
- added link eef_link, mass 0.001
Joints:
- added joint fix_linear_rail_and_end_effector: type fixed, parent linear_rail, child eef_link, origin xyz=0.14 0 0 rpy=0 0 0

Commit message: feature: remove mirror

File: urdf/umi_gripper/umi_gripper.urdf (robot description, URDF)
Before this commit: robot umi_gripper, 22 links, 21 joints
Links:
- removed link left_mirror
- removed link right_mirror
Joints:
- removed joint fix_linear_rail_and_left_mirror
- removed joint fix_linear_rail_and_right_mirror

Commit message: test: 修改镜头位置

File: urdf/umi_gripper/umi_gripper.urdf (robot description, URDF)
Before this commit: robot umi_gripper, 22 links, 21 joints
Joints:
- joint fix_linear_rail_and_gopro: origin xyz=-0.0522 0.0 0.09 rpy=0 0 0 -> xyz=-0.0552 0.0 0.087 rpy=0 0 0
