Commit message: feature: change to a2-vx300s-umi

File: urdf/a2-vx300s/a2-vx300s.urdf (robot description, URDF)
Before this commit: robot a2_vx300s, 30 links, 29 joints
Links:
- added link gopro, mass 0.127; visual mesh filename=meshes/gopro.stl scale=1 1 1
- link vx300s_left_finger_link: mass 0.034796 -> 0.043; geometry collision mesh filename=meshes/umi_left_finger_collision.stl scale=1 1 1; visual mesh filename=meshes/umi_left_finger.stl scale=1 1 1
- link vx300s_right_finger_link: mass 0.034796 -> 0.043; geometry collision mesh filename=meshes/umi_right_finger_collision.stl scale=1 1 1; visual mesh filename=meshes/umi_right_finger.stl scale=1 1 1
Joints:
- added joint joint_gopro: type fixed, parent vx300s_fingers_link, child gopro, origin xyz=-0.0522 0.0 0.09 rpy=0 0 0, axis 0 1 0
- joint fix_eef_link: origin xyz=0.0385 0 0 rpy=0 0 0 -> xyz=0.14 0 0 rpy=0 0 0
- joint left_finger_joint: limit lower=0 upper=0.036 effort=5 velocity=1 -> lower=0 upper=0.0425 effort=10 velocity=0.1; origin xyz=0 0.0085 0 rpy=0 0 0 -> xyz=0 0 0 rpy=0 0 0
- joint right_finger_joint: limit lower=0 upper=0.036 effort=5 velocity=1 -> lower=0 upper=0.0425 effort=10 velocity=0.1; origin xyz=0 -0.0085 0 rpy=0 0 0 -> xyz=0 0 0 rpy=0 0 0

Commit message: test: 修改镜头位置

File: urdf/a2-vx300s/a2-vx300s.urdf (robot description, URDF)
Before this commit: robot a2_vx300s, 39 links, 38 joints
Joints:
- joint joint_gopro: origin xyz=-0.0522 0.0 0.09 rpy=0 0 0 -> xyz=-0.0552 0.0 0.087 rpy=0 0 0
